File: FLIM 4-1 Mux controller/FLIM 4-1 Mux controller.kicad_sch (KiCad schematic)
At the start: 20 parts, among them J1 Conn_01x14_Pin, J10 Conn_01x03_Socket, J11 Conn_01x03_Pin, J12 Conn_01x03_Socket, J2 Conn_01x14_Pin, J3 Conn_01x05_Pin, J4 RJ45_Shielded, J5 Conn_01x03_Pin, J6 Conn_01x03_Socket, J7 Conn_01x03_Pin, J8 Conn_01x03_Socket, J9 Conn_01x03_Pin, SW1 SW_Push_LED, SW2 SW_Push_LED, SW3 SW_Push_LED, SW4 SW_Push_LED, U1 Itsy_Bitsy_32u4

Commit message: Finished working draft of PCB - passes DRC
Parts:
- removed RN1: 1k, Resistor_SMD:R_Array_Convex_4x0603, symbol Device:R_Pack04
- added RN3: 1k, Resistor_SMD:R_Array_Convex_4x0603, symbol Device:R_Pack04
Connections:
- net CLK: now also RN3.5 (R4.2)
- net CLK*: now also RN3.4 (R4.1)
- net D1: now also RN3.8 (R1.2)
- net D1*: now also RN3.1 (R1.1)
- net D2: now also RN3.7 (R2.2)
- net D2*: now also RN3.2 (R2.1)
- net D3: now also RN3.6 (R3.2)
- net D3*: now also RN3.3 (R3.1)
Changed lines of the file:
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@@
 	(symbol
 		(lib_id "Device:R_Pack04")
-		(at 39.37 143.51 90)
+		(at 39.37 146.05 90)
+		(mirror x)
 		(unit 1)
 		(body_style 1)
@@
 		(in_pos_files yes)
 		(dnp no)
-		(fields_autoplaced yes)
-		(property "Reference" "RN1"
-			(at 39.37 135.5555 90)
+		(property "Reference" "RN3"
+			(at 39.37 136.652 90)
 			(show_name no)
 			(do_not_autoplace no)
@@
 		)
 		(property "Value" "1k"
-			(at 39.37 137.9798 90)
+			(at 39.37 138.684 90)
 			(show_name no)
 			(do_not_autoplace no)
@@
 		)
 		(property "Footprint" "Resistor_SMD:R_Array_Convex_4x0603"
-			(at 39.37 136.525 90)
+			(at 39.37 153.035 90)
 			(hide yes)
 			(show_name no)
@@
 			)
 		)
-		(property "Datasheet" "https://www.seielect.com/catalog/SEI-RAVF.pdf"
-			(at 39.37 143.51 0)
+		(property "Datasheet" "https://www.bourns.com/docs/Product-Datasheets/CATCAY.pdf"
+			(at 39.37 146.05 0)
 			(hide yes)
 			(show_name no)
@@
 			)
 		)
-		(property "Description" "1k Ohm ±5% 100mW Power Per Element Isolated 4 Resistor Network/Array ±200ppm/°C 1206 (3216 Metric), Convex, Long Side Terminals"
-			(at 39.37 143.51 0)
+		(property "Description" "22k Ohm ±1% 62.5mW Power Per Element Isolated 4 Resistor Network/Array ±200ppm/°C 1206 (3216 Metric), Convex, Long Side Terminals"
+			(at 39.37 146.05 0)
 			(hide yes)
 			(show_name no)
@@
 			)
 		)
-		(property "Manufacturer" "Stackpole Electronics Inc"
-			(at 39.37 143.51 0)
+		(property "Manufacturer" "Bourns Inc."
+			(at 39.37 146.05 0)
 			(hide yes)
 			(show_name no)
@@
 			)
 		)
-		(property "Part #" "RAVF164DJT1K00"
-			(at 39.37 143.51 90)
+		(property "Part #" "CAY16-1001F4LF"
+			(at 39.37 146.05 90)
 			(hide yes)
 			(show_name no)
@@
 			(project "FLIM 4-1 Mux controller"
 				(path "/9a5ec920-9f12-407d-b06b-b123ad2c0d9b"
-					(reference "RN1")
+					(reference "RN3")
 					(unit 1)
 				)
