File: FLIM 4-1 Mux board/FLIM 4-1 Mux board.kicad_sch (KiCad schematic)
At the start: 62 parts, among them J1 Barrel_Jack, J2 RJ45_Shielded, J3 Conn_Coaxial, J4 Conn_Coaxial, J5 Conn_Coaxial, J6 Conn_Coaxial, J7 Conn_Coaxial, U1 ADM7150ARDZ-5.0, U2 74AHCT74D_118, U3 74AHCT74D_118, U4 SPDT RF switch, U5 SPDT RF switch, U6 SPDT RF switch

Commit message: Shorten SMA pins to reduce impedance mismatch at 4GHz, add standoffs and enclosure
Parts:
- added H1, H2, H3, H4: (no value), Custom:MountingHole_4.3mm_M4_Pad_Via, symbol Mechanical:MountingHole_Pad
- added N1: Housing_Pad, symbol Mechanical:Housing_Pad
Connections:
- net GND: now also H1.1, H2.1, H3.1, H4.1, N1.1 (PAD)

Commit message: Switch to 100 nF 0201 RF caps for waveguides
Parts:
- C19, C26, C27, C28, C29, C30, C31: value 8.2 nF -> 100 nF; footprint Capacitor_SMD:C_0402_1005Metric -> Capacitor_SMD:C_0201_0603Metric; Manufacturer Murata Electronics -> Passive Plus; Part # GRM1555C1H822GE01D -> 0201BB104KW160
Connections:
- net at J3.1 (In): now also C19.2; no longer C19.1
- net at U4.3 (RFC): now also C19.1; no longer C19.2
